Commit message: robot no turning

File: description/robot_core.xacro (robot description, xacro)
@@ -57,32 +57,12 @@
         </xacro:inertial_box>
     </link>
-<!-- left wheel link-->
-    <joint name="left_wheel_joint" type="continuous">
-        <parent link="base_link"/>
-        <child link="left_wheel"/>
-        <origin xyz="0.0 0.27 0.0" rpy="-${pi/2} 0.0 0.0"/>
-        <axis xyz="0.0 0.0 1"/>
-    </joint>
-    <link name="left_wheel">
-        <visual>
-            <geometry>
-                <cylinder radius="0.1" length="0.04"/>
-            </geometry>
-            <material name="blue"/>
-        </visual>
-        <collision>
-            <geometry>
-                <cylinder radius="0.1" length="0.04"/>
-            </geometry>
-        </collision>
-        <xacro:inertial_cylinder mass="0.1" length="0.04" radius="0.1" >
-            <origin xyz="0.0 0.0 0.0" rpy="0.0 0.0 0.0"/>
-        </xacro:inertial_cylinder>
-    </link>
+    <gazebo reference="chassis">
+        <material>Gazebo/White</material>
+    </gazebo>
 <!-- right wheel link-->
     <joint name="right_wheel_joint" type="continuous">
         <parent link="base_link"/>
         <child link="right_wheel"/>
-        <origin xyz="0.0 -0.27 0.0" rpy="${pi/2} 0.0 0.0"/>
+        <origin xyz="0.0 0.27 0.0" rpy="-${pi/2} 0.0 0.0"/>
         <axis xyz="0.0 0.0 -1"/>
     </joint>
@@ -103,4 +83,49 @@
         </xacro:inertial_cylinder>
     </link>
+    <gazebo reference="right_wheel">
+        <material>Gazebo/Blue</material>
+        <surface>
+            <friction>
+                <ode>
+                    <mu1>1.0</mu1>
+                    <mu2>1.0</mu2>
+                </ode>
+            </friction>
+        </surface>
+    </gazebo>
+<!-- left wheel link-->
+    <joint name="left_wheel_joint" type="continuous">
+        <parent link="base_link"/>
+        <child link="left_wheel"/>
+        <origin xyz="0 -0.27 0" rpy="${pi/2} 0 0"/>
+        <axis xyz="0 0 1"/>
+    </joint>
+    <link name="left_wheel">
+        <visual>
+            <geometry>
+                <cylinder radius="0.1" length="0.04"/>
+            </geometry>
+            <material name="blue"/>
+        </visual>
+        <collision>
+            <geometry>
+                <cylinder radius="0.1" length="0.04"/>
+            </geometry>
+        </collision>
+        <xacro:inertial_cylinder mass="0.1" length="0.04" radius="0.1" >
+            <origin xyz="0 0 0" rpy="0 0 0"/>
+        </xacro:inertial_cylinder>
+    </link>
+    <gazebo reference="left_wheel">
+        <material>Gazebo/Blue</material>
+        <surface>
+            <friction>
+                <ode>
+                    <mu>1</mu>
+                    <mu2>1</mu2>
+                </ode>
+            </friction>
+        </surface>
+    </gazebo>
 <!-- caster wheel link-->
     <joint name="caster_wheel_joint" type="fixed">
@@ -121,7 +146,20 @@
             </geometry>
         </collision>
-        <xacro:inertial_sphere mass="0.1" radius="0.5" >
+        <xacro:inertial_sphere mass="0.1" radius="0.05" >
             <origin xyz="0.0 0.0 0.0" rpy="0.0 0.0 0.0"/>
         </xacro:inertial_sphere>
     </link>
+    <gazebo reference="caster_wheel">
+        <material>Gazebo/Black</material>
+        <surface>
+            <friction>
+                <ode>
+                    <mu>0.0001</mu>
+                    <mu2>0.0001</mu2>
+                    <slip1>0.1</slip1>
+                    <slip2>0.1</slip2>
+                </ode>
+            </friction>
+        </surface>
+    </gazebo>
 </robot>

Commit message: gazebo basic done

File: description/robot_core.xacro (robot description, xacro)
@@ -50,9 +50,6 @@
             </geometry>
         </collision>
-        <xacro:inertial_box mass="0.5" x="0.75" y="0.1" z="0.03" >
-            <origin xyz="0.0 0.0 0.0" rpy="0 0 0"/>
-        </xacro:inertial_box>
-        <xacro:inertial_box mass="0.5" x="0.1" y="0.5" z="0.03" >
-            <origin xyz="-0.35 0.0 0.0" rpy="0 0 0"/>
+        <xacro:inertial_box mass="0.5" x="0.75" y="0.5" z="0.03" >
+            <origin xyz="0 0.0 0.0" rpy="0 0 0"/>
         </xacro:inertial_box>
     </link>
@@ -65,5 +62,5 @@
         <child link="right_wheel"/>
         <origin xyz="0.0 0.27 0.0" rpy="-${pi/2} 0.0 0.0"/>
-        <axis xyz="0.0 0.0 -1"/>
+        <axis xyz="0.0 0.0 1"/>
     </joint>
     <link name="right_wheel">
@@ -85,12 +82,4 @@
     <gazebo reference="right_wheel">
         <material>Gazebo/Blue</material>
-        <surface>
-            <friction>
-                <ode>
-                    <mu1>1.0</mu1>
-                    <mu2>1.0</mu2>
-                </ode>
-            </friction>
-        </surface>
     </gazebo>
 <!-- left wheel link-->
@@ -99,5 +88,5 @@
         <child link="left_wheel"/>
         <origin xyz="0 -0.27 0" rpy="${pi/2} 0 0"/>
-        <axis xyz="0 0 1"/>
+        <axis xyz="0 0 -1"/>
     </joint>
     <link name="left_wheel">
@@ -119,12 +108,4 @@
     <gazebo reference="left_wheel">
         <material>Gazebo/Blue</material>
-        <surface>
-            <friction>
-                <ode>
-                    <mu>1</mu>
-                    <mu2>1</mu2>
-                </ode>
-            </friction>
-        </surface>
     </gazebo>
 <!-- caster wheel link-->
@@ -152,14 +133,6 @@
     <gazebo reference="caster_wheel">
         <material>Gazebo/Black</material>
-        <surface>
-            <friction>
-                <ode>
-                    <mu>0.0001</mu>
-                    <mu2>0.0001</mu2>
-                    <slip1>0.1</slip1>
-                    <slip2>0.1</slip2>
-                </ode>
-            </friction>
-        </surface>
+        <mu1 value="0.001"/>
+        <mu2 value="0.001"/>
     </gazebo>
 </robot>
